File: hw/oratio-pcb-1/oratio-pcb-1.kicad_sch (KiCad schematic)
At the start: 0 parts

Commit message: initial layout of components in schematic AB#166
Parts:
- added D1, D2, D3: LED, LED_THT:LED_D3.0mm, symbol Device:LED
- added SW1: SW_SPST, Button_Switch_THT:SW_PUSH_6mm_H5mm, symbol Switch:SW_SPST
- added U1: ESP32-S3-DevKitC, PCM_Espressif:ESP32-S3-DevKitC, symbol PCM_Espressif:ESP32-S3-DevKitC
- added U2: INMP441 BREAKOUT, symbol oratio:INMP441_Breakout
- added U3: MAX98357A BREAKOUT, symbol oratio:MAX98357A_Breakout
Connections:
- new net: U1.1 (3V3), U1.2 (3V3)
- new net: U1.22 (GND), U1.23 (GND), U1.24 (GND), U1.44 (GND)
Other:
- company: (none) -> Oratio

Commit message: initial routing of schematic AB#166
Parts:
- added R1, R2, R3: 330R, Resistor_THT:R_Axial_DIN0207_L6.3mm_D2.5mm_P10.16mm_Horizontal, symbol Device:R_US
Connections:
- net +3.3V: now reaches U1.1 (3V3), U1.2 (3V3)
- net +3.3V: now also U2.2 (VDD)
- net +5V: now reaches U1.21 (5V)
- net GND: now reaches U1.22 (GND), U1.23 (GND), U1.24 (GND), U1.44 (GND)
- net GND: now also SW1.2 (B), U2.1 (GND), U2.4 (L/R), U3.6 (GND), R1.2, R2.2, R3.2
- net PTT_GPIO: now reaches U1.27 (GPIO21)
- net PTT_GPIO: now also SW1.1 (A)
- net SPK_WS: now reaches U3.1 (LRC)
- net SPK_SCK: now reaches U3.2 (BCLK)
- net SPK_DIN: now reaches U3.3 (DIN)
- net at D2.1 (K): now also R2.1
- net LED2_GPIO: now reaches D2.2 (A)
- net at D1.1 (K): now also R1.1
- net LED1_GPIO: now reaches D1.2 (A)
- net MIC_SD: now reaches U2.3 (SD)
- net MIC_WS: now reaches U2.5 (WS)
- net MIC_SCK: now reaches U2.6 (SCK)
- net at D3.1 (K): now also R3.1
- net LED3_GPIO: now reaches D3.2 (A)
Other:
- moved on the sheet: D1, D2, D3, SW1
